File: kicad-pcb-force-sensor/kicad-pcb-force-sensor.kicad_sch (KiCad schematic)
At the start: 17 parts, among them J1 Power, J2 Digital/PWM, J3 Analog, J4 Digital/PWM, U3 KY-040

Commit message: flex_sensor
Parts:
- added Flex_sensor1: ~, graphite_emprunts:Flex, symbol graphite_library:Flex_Sensor
- added Rflex1: 23k, Resistor_THT:R_Axial_DIN0207_L6.3mm_D2.5mm_P10.16mm_Horizontal, symbol Device:R
Connections:
- net GND: now also Rflex1.2
- net VCC: now also Flex_sensor1.1 (+)
- net A1 renamed Flex
- net Flex: now also Flex_sensor1.2 (-), Rflex1.1
Other:
- moved on the sheet: Ecran1, Pot_Digital1

Commit message: Servo
Parts:
- added M1: Motor_Servo, graphite_emprunts:Servo, symbol Motor:Motor_Servo
Connections:
- net GND: now also M1.3 (-)
- net VCC: now also M1.2 (+)
- net D9 renamed D9 PWM
- net D9 PWM: now also M1.1 (PWM)
Other:
- moved on the sheet: Flex_sensor1, Rflex1
Changed lines of the file:
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@@
 	)
 	(junction
-		(at 176.53 106.68)
+		(at 146.05 114.3)
 		(diameter 0)
 		(color 0 0 0 0)
@@
 	(wire
 		(pts
+			(xy 173.99 111.76) (xy 177.8 111.76)
+		)
+		(stroke
+			(width 0)
+			(type default)
+		)
+	)
+	(wire
+		(pts
 			(xy 62.23 26.67) (xy 74.93 26.67)
 		)
@@
 	(wire
 		(pts
-			(xy 170.18 102.87) (xy 173.99 102.87)
+			(xy 139.7 110.49) (xy 143.51 110.49)
 		)
 		(stroke
@@
 	(wire
 		(pts
-			(xy 62.23 46.99) (xy 74.93 46.99)
+			(xy 62.23 46.99) (xy 81.28 46.99)
 		)
 		(stroke
@@
 	(wire
 		(pts
-			(xy 181.61 106.68) (xy 176.53 106.68)
+			(xy 151.13 114.3) (xy 146.05 114.3)
 		)
 		(stroke
@@
 	(wire
 		(pts
+			(xy 173.99 109.22) (xy 177.8 109.22)
+		)
+		(stroke
+			(width 0)
+			(type default)
+		)
+	)
+	(wire
+		(pts
 			(xy 19.05 72.39) (xy 34.29 72.39)
 		)
@@
 	(wire
 		(pts
-			(xy 176.53 115.57) (xy 176.53 121.92)
+			(xy 146.05 123.19) (xy 146.05 129.54)
 		)
 		(stroke
@@
 	(wire
 		(pts
-			(xy 176.53 106.68) (xy 176.53 107.95)
+			(xy 146.05 114.3) (xy 146.05 115.57)
 		)
 		(stroke
@@
 	(wire
 		(pts
-			(xy 173.99 100.33) (xy 173.99 102.87)
+			(xy 143.51 107.95) (xy 143.51 110.49)
 		)
 		(stroke
@@
 	(wire
 		(pts
+			(xy 172.72 114.3) (xy 177.8 114.3)
+		)
+		(stroke
+			(width 0)
+			(type default)
+		)
+	)
+	(wire
+		(pts
 			(xy 69.85 189.23) (xy 69.85 191.77)
 		)
@@
 	(wire
 		(pts
-			(xy 176.53 100.33) (xy 176.53 106.68)
+			(xy 146.05 107.95) (xy 146.05 114.3)
 		)
 		(stroke
@@
 	(wire
 		(pts
-			(xy 62.23 49.53) (xy 82.55 49.53)
+			(xy 62.23 49.53) (xy 81.28 49.53)
 		)
 		(stroke
@@
 	(global_label "Flex"
 		(shape input)
-		(at 181.61 106.68 0)
+		(at 151.13 114.3 0)
 		(fields_autoplaced yes)
 		(effects
@@
 		)
 		(property "Intersheetrefs" "${INTERSHEET_REFS}"
-			(at 188.5608 106.68 0)
+			(at 158.0808 114.3 0)
 			(effects
 				(font
@@
 		)
 	)
+	(global_label "D9 PWM"
+		(shape input)
+		(at 81.28 46.99 0)
+		(fields_autoplaced yes)
+		(effects
+			(font
+				(size 1.27 1.27)
+			)
+			(justify left)
+		)
+		(property "Intersheetrefs" "${INTERSHEET_REFS}"
+			(at 91.9802 46.99 0)
+			(effects
+				(font
+					(size 1.27 1.27)
+				)
+				(justify left)
+				(hide yes)
+			)
+		)
+	)
 	(global_label "RXD"
 		(shape input)
@@
 	(global_label "VCC"
 		(shape input)
-		(at 170.18 102.87 180)
+		(at 173.99 111.76 180)
 		(fields_autoplaced yes)
 		(effects
@@
 		)
 		(property "Intersheetrefs" "${INTERSHEET_REFS}"
-			(at 163.4711 102.87 0)
+			(at 167.2811 111.76 0)
+			(effects
+				(font
+					(size 1.27 1.27)
+				)
+				(justify right)
+				(hide yes)
+			)
+		)
+	)
+	(global_label "VCC"
+		(shape input)
+		(at 139.7 110.49 180)
+		(fields_autoplaced yes)
+		(effects
+			(font
+				(size 1.27 1.27)
+			)
+			(justify right)
+		)
+		(property "Intersheetrefs" "${INTERSHEET_REFS}"
+			(at 132.9911 110.49 0)
 			(effects
 				(font
@@
 		)
 	)
+	(global_label "GND"
+		(shape input)
+		(at 172.72 114.3 180)
+		(fields_autoplaced yes)
+		(effects
+			(font
+				(size 1.27 1.27)
+			)
+			(justify right)
+		)
+		(property "Intersheetrefs" "${INTERSHEET_REFS}"
+			(at 165.7692 114.3 0)
+			(effects
+				(font
+					(size 1.27 1.27)
+				)
+				(justify right)
+				(hide yes)
+			)
+		)
+	)
 	(global_label "VCC"
 		(shape input)
@@
 		)
 	)
+	(global_label "D9 PWM"
+		(shape input)
+		(at 173.99 109.22 180)
+		(fields_autoplaced yes)
+		(effects
+			(font
+				(size 1.27 1.27)
+			)
+			(justify right)
+		)
+		(property "Intersheetrefs" "${INTERSHEET_REFS}"
+			(at 163.2898 109.22 0)
+			(effects
+				(font
+					(size 1.27 1.27)
+				)
+				(justify right)
+				(hide yes)
+			)
+		)
+	)
 	(global_label "SDA"
 		(shape input)
@@
 	(global_label "TXD"
 		(shape input)
-		(at 82.55 49.53 0)
+		(at 81.28 49.53 0)
 		(fields_autoplaced yes)
 		(effects
@@
 		)
 		(property "Intersheetrefs" "${INTERSHEET_REFS}"
-			(at 89.0774 49.53 0)
+			(at 87.8074 49.53 0)
 			(effects
 				(font
@@
 	(global_label "GND"
 		(shape input)
-		(at 176.53 121.92 270)
+		(at 146.05 129.54 270)
 		(fields_autoplaced yes)
 		(effects
@@
 		)
 		(property "Intersheetrefs" "${INTERSHEET_REFS}"
-			(at 176.53 128.8708 90)
+			(at 146.05 136.4908 90)
 			(effects
 				(font
@@
 	(symbol
 		(lib_id "graphite_library:Flex_Sensor")
-		(at 175.26 100.33 0)
+		(at 144.78 107.95 0)
 		(unit 1)
 		(exclude_from_sim no)
@@
 		(fields_autoplaced yes)
 		(property "Reference" "Flex_sensor1"
-			(at 177.8 95.2499 0)
+			(at 147.32 102.8699 0)
 			(effects
 				(font
@@
 		)
 		(property "Value" "~"
-			(at 177.8 97.7899 0)
+			(at 147.32 105.4099 0)
 			(effects
 				(font
@@
 		)
 		(property "Footprint" "graphite_emprunts:Flex"
-			(at 175.26 100.33 0)
+			(at 144.78 107.95 0)
 			(effects
 				(font
@@
 		)
 		(property "Datasheet" ""
-			(at 175.26 100.33 0)
+			(at 144.78 107.95 0)
 			(effects
 				(font
@@
 		)
 		(property "Description" ""
-			(at 175.26 100.33 0)
+			(at 144.78 107.95 0)
 			(effects
 				(font
@@
 	)
 	(symbol
+		(lib_id "Motor:Motor_Servo")
+		(at 185.42 111.76 0)
+		(unit 1)
+		(exclude_from_sim no)
+		(in_bom yes)
+		(on_board yes)
+		(dnp no)
+		(fields_autoplaced yes)
+		(property "Reference" "M1"
+			(at 194.31 110.0568 0)
+			(effects
+				(font
+					(size 1.27 1.27)
+				)
+				(justify left)
+			)
+		)
+		(property "Value" "Motor_Servo"
+			(at 194.31 112.5968 0)
+			(effects
+				(font
+					(size 1.27 1.27)
+				)
+				(justify left)
+			)
+		)
+		(property "Footprint" "graphite_emprunts:Servo"
+			(at 185.42 116.586 0)
+			(effects
+				(font
+					(size 1.27 1.27)
+				)
+				(hide yes)
+			)
+		)
+		(property "Datasheet" ""
+			(at 185.42 116.586 0)
+			(effects
+				(font
+					(size 1.27 1.27)
+				)
+				(hide yes)
+			)
+		)
+		(property "Description" "Servo Motor (Futaba, HiTec, JR connector)"
+			(at 185.42 111.76 0)
+			(effects
+				(font
+					(size 1.27 1.27)
+				)
+				(hide yes)
+			)
+		)
+		(pin "2"
+		)
+		(pin "3"
+		)
+		(pin "1"
+		)
+		(instances
+			(project ""
+				(path "/e63e39d7-6ac0-4ffd-8aa3-1841a4541b55"
+					(reference "M1")
+					(unit 1)
+				)
+			)
+		)
+	)
+	(symbol
 		(lib_id "graphite_library:KY-040")
 		(at 127 86.36 0)
@@
 	(symbol
 		(lib_id "Device:R")
-		(at 176.53 111.76 0)
+		(at 146.05 119.38 0)
 		(unit 1)
 		(exclude_from_sim no)
@@
 		(fields_autoplaced yes)
 		(property "Reference" "Rflex1"
-			(at 179.07 110.4899 0)
+			(at 148.59 118.1099 0)
 			(effects
 				(font
@@
 		)
 		(property "Value" "23k"
-			(at 179.07 113.0299 0)
+			(at 148.59 120.6499 0)
 			(effects
 				(font
@@
 		)
 		(property "Footprint" "Resistor_THT:R_Axial_DIN0207_L6.3mm_D2.5mm_P10.16mm_Horizontal"
-			(at 174.752 111.76 90)
+			(at 144.272 119.38 90)
 			(effects
 				(font
@@
 		)
 		(property "Datasheet" "~"
-			(at 176.53 111.76 0)
+			(at 146.05 119.38 0)
 			(effects
 				(font
@@
 		)
 		(property "Description" "Resistor"
-			(at 176.53 111.76 0)
+			(at 146.05 119.38 0)
 			(effects
 				(font
