File: kicad-pcb-force-sensor/kicad-pcb-force-sensor.kicad_sch (KiCad schematic)
At the start: 20 parts, among them J1 Power, J2 Digital/PWM, J3 Analog, J4 Digital/PWM, M1 Motor_Servo, U3 KY-040

Commit message: Avec pistes
Connections:
- net D10 PWM/MOSI is gone; now on net D10 PWM/SS: J2.8 (Pin_8)
Changed lines of the file:
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@@
 		)
 	)
-	(global_label "D10 PWM{slash}MOSI"
+	(global_label "D10 PWM{slash}SS"
 		(shape input)
 		(at 81.28 44.45 0)
@@
 		)
 		(property "Intersheetrefs" "${INTERSHEET_REFS}"
-			(at 99.1164 44.45 0)
+			(at 96.9392 44.45 0)
 			(effects
 				(font

Commit message: Modifier pins à 0.8mm plus détails
Parts:
- Rflex1: value 23k -> 47k
Changed lines of the file:
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@@
 			)
 		)
-		(property "Value" "23k"
+		(property "Value" "47k"
 			(at 148.59 120.6499 0)
 			(effects

Commit message: partie Kicad
Parts:
- renumbered Ecran1 to DM-OLED096-636
Connections:
- net ADC is gone; now on net GND: C2.2, J3.1 (Pin_1), R6.2
- net GND: now also AOP1.3 (+IN), C1.2, R1.1, R5.2
Other:
- moved on the sheet: AOP1, C1, C2, C4, DM-OLED096-636, Flex_sensor1, Graphite_sensor1, J1, J2, J3, J4, M1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

Commit message: Caractérisation et datasheet
Other:
- title: Flex Sensor board  -> PROJET MOSH
Changed lines of the file:
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@@
 	(paper "A4")
 	(title_block
-		(title "Flex Sensor board ")
+		(title "PROJET MOSH")
 		(date "2026-02-10")
 		(rev "${VERSION_NUMBER}")

Commit message: nueva datasheet
Parts:
- R3: value 1k -> 100k
Changed lines of the file:
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@@
 			)
 		)
-		(property "Value" "1k"
+		(property "Value" "100k"
 			(at 242.57 55.8799 0)
 			(effects
