File: kicad-pcb-force-sensor/kicad-pcb-force-sensor.kicad_pcb (KiCad board)
At the start: 2 copper layers, 68.6 x 53.3 mm, 22 parts, among them J1 Power, J2 Digital/PWM, J3 Analog, J4 Digital/PWM, U3 KY-040

Commit message: Pines graphic sesor
Connections:
- AOP1 pad 7: R2 -> VCC
- Ecran1 pad 2: R2 -> VCC
- Graphite_sensor1 pad 1: unconnected-(Graphite_sensor1-+-Pad1) -> VCC
- Graphite_sensor1 pad 2: unconnected-(Graphite_sensor1---Pad2) -> Net-(Graphite_sensor1--)
- J1 pad 8: R2 -> VCC
- Pot_Digital1 pad 5: R2 -> Net-(Pot_Digital1-PA0)
- Pot_Digital1 pad 6: unconnected-(Pot_Digital1-PW0-Pad6) -> Net-(Pot_Digital1-PA0)
- Pot_Digital1 pad 7: GND -> R2
- Pot_Digital1 pad 8: R2 -> VCC
- R5 pad 1: unconnected-(R5-Pad1) -> Net-(Graphite_sensor1--)
- U1 pad 1: R2 -> VCC
- U3 pad VCC: R2 -> VCC
Changed lines of the file:
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@@
 	(net 11 "/RX{slash}0")
 	(net 12 "+3V3")
-	(net 13 "unconnected-(Pot_Digital1-PW0-Pad6)")
+	(net 13 "VCC")
 	(net 14 "/~{RESET}")
 	(net 15 "/D12")
 	(net 16 "/D9")
 	(net 17 "ADC")
-	(net 18 "unconnected-(R5-Pad1)")
+	(net 18 "Net-(Graphite_sensor1--)")
 	(net 19 "TXD")
 	(net 20 "RXD")
@@
 	(net 32 "R2")
 	(net 33 "D10 PWM{slash}SS")
-	(net 34 "unconnected-(Graphite_sensor1-+-Pad1)")
-	(net 35 "unconnected-(Graphite_sensor1---Pad2)")
-	(net 36 "Net-(AOP1-OUT)")
-	(net 37 "Net-(AOP1--IN)")
-	(net 38 "unconnected-(AOP1-NC-Pad8)")
-	(net 39 "unconnected-(AOP1-NC_2-Pad1)")
-	(net 40 "unconnected-(AOP1-EXTCLOCKINPUT-Pad5)")
-	(net 41 "Net-(AOP1-+IN)")
+	(net 34 "Net-(Pot_Digital1-PA0)")
+	(net 35 "Net-(AOP1-OUT)")
+	(net 36 "Net-(AOP1--IN)")
+	(net 37 "unconnected-(AOP1-NC-Pad8)")
+	(net 38 "unconnected-(AOP1-NC_2-Pad1)")
+	(net 39 "unconnected-(AOP1-EXTCLOCKINPUT-Pad5)")
+	(net 40 "Net-(AOP1-+IN)")
 	(footprint "Connector_PinSocket_2.54mm:PinSocket_1x08_P2.54mm_Vertical"
 		(locked yes)
@@
 			)
 		)
-		(property "Datasheet" "~"
+		(property "Datasheet" ""
 			(at 0 0 90)
 			(unlocked yes)
@@
 			(layers "*.Cu" "*.Mask")
 			(remove_unused_layers no)
-			(net 32 "R2")
+			(net 13 "VCC")
 			(pinfunction "Pin_8")
 			(pintype "passive")
@@
 			)
 		)
-		(property "Datasheet" "~"
+		(property "Datasheet" ""
 			(at 0 0 90)
 			(unlocked yes)
@@
 			)
 		)
-		(property "Datasheet" "~"
+		(property "Datasheet" ""
 			(at 0 0 90)
 			(unlocked yes)
@@
 			)
 		)
-		(property "Datasheet" "~"
+		(property "Datasheet" ""
 			(at 0 0 90)
 			(unlocked yes)
@@
 			(layers "*.Cu" "*.Mask")
 			(remove_unused_layers no)
-			(net 39 "unconnected-(AOP1-NC_2-Pad1)")
+			(net 38 "unconnected-(AOP1-NC_2-Pad1)")
 			(pinfunction "NC_2")
 			(pintype "no_connect")
@@
 			(layers "*.Cu" "*.Mask")
 			(remove_unused_layers no)
-			(net 41 "Net-(AOP1-+IN)")
+			(net 40 "Net-(AOP1-+IN)")
 			(pinfunction "+IN")
 			(pintype "input")
@@
 			(layers "*.Cu" "*.Mask")
 			(remove_unused_layers no)
-			(net 40 "unconnected-(AOP1-EXTCLOCKINPUT-Pad5)")
+			(net 39 "unconnected-(AOP1-EXTCLOCKINPUT-Pad5)")
 			(pinfunction "EXTCLOCKINPUT")
 			(pintype "no_connect")
@@
 			(layers "*.Cu" "*.Mask")
 			(remove_unused_layers no)
-			(net 36 "Net-(AOP1-OUT)")
+			(net 35 "Net-(AOP1-OUT)")
 			(pinfunction "OUT")
 			(pintype "output")
@@
 			(layers "*.Cu" "*.Mask")
 			(remove_unused_layers no)
-			(net 32 "R2")
+			(net 13 "VCC")
 			(pinfunction "V+")
 			(pintype "power_in")
@@
 			(layers "*.Cu" "*.Mask")
 			(remove_unused_layers no)
-			(net 38 "unconnected-(AOP1-NC-Pad8)")
+			(net 37 "unconnected-(AOP1-NC-Pad8)")
 			(pinfunction "NC")
 			(pintype "no_connect")
@@
 			(layers "*.Cu" "*.Mask")
 			(remove_unused_layers no)
-			(net 37 "Net-(AOP1--IN)")
+			(net 36 "Net-(AOP1--IN)")
 			(pintype "passive")
 		)
@@
 			(layers "*.Cu" "*.Mask")
 			(remove_unused_layers no)
-			(net 32 "R2")
+			(net 13 "VCC")
 			(pinfunction "VCC")
 			(pintype "power_in")
@@
 			(layers "*.Cu" "*.Mask")
 			(remove_unused_layers no)
-			(net 32 "R2")
+			(net 13 "VCC")
 			(pinfunction "VCC_IN")
 			(pintype "power_in")
@@
 			(layers "*.Cu" "*.Mask")
 			(remove_unused_layers no)
-			(net 34 "unconnected-(Graphite_sensor1-+-Pad1)")
+			(net 13 "VCC")
 			(pinfunction "+")
 			(pintype "input")
@@
 			(layers "*.Cu" "*.Mask")
 			(remove_unused_layers no)
-			(net 35 "unconnected-(Graphite_sensor1---Pad2)")
+			(net 18 "Net-(Graphite_sensor1--)")
 			(pinfunction "-")
 			(pintype "input")
@@
 			(layers "*.Cu" "*.Mask")
 			(remove_unused_layers no)
-			(net 32 "R2")
+			(net 13 "VCC")
 			(pinfunction "Vcc")
 			(pintype "input")
@@
 			)
 		)
-		(property "Datasheet" "~"
+		(property "Datasheet" ""
 			(at 0 0 0)
 			(layer "F.Fab")
@@
 			(layers "*.Cu" "*.Mask")
 			(remove_unused_layers no)
-			(net 41 "Net-(AOP1-+IN)")
+			(net 40 "Net-(AOP1-+IN)")
 			(pintype "passive")
 		)
@@
 			)
 		)
-		(property "Datasheet" "~"
+		(property "Datasheet" ""
 			(at 0 0 0)
 			(layer "F.Fab")
@@
 			(layers "*.Cu" "*.Mask")
 			(remove_unused_layers no)
-			(net 41 "Net-(AOP1-+IN)")
+			(net 40 "Net-(AOP1-+IN)")
 			(pintype "passive")
 		)
@@
 			)
 		)
-		(property "Datasheet" "~"
+		(property "Datasheet" ""
 			(at 0 0 0)
 			(layer "F.Fab")
@@
 			(layers "*.Cu" "*.Mask")
 			(remove_unused_layers no)
-			(net 18 "unconnected-(R5-Pad1)")
+			(net 18 "Net-(Graphite_sensor1--)")
 			(pintype "passive")
 		)
@@
 			(layers "*.Cu" "*.Mask")
 			(remove_unused_layers no)
-			(net 41 "Net-(AOP1-+IN)")
+			(net 40 "Net-(AOP1-+IN)")
 			(pintype "passive")
 		)
@@
 			)
 		)
-		(property "Datasheet" "~"
+		(property "Datasheet" ""
 			(at 0 0 0)
 			(layer "F.Fab")
@@
 			(layers "*.Cu" "*.Mask")
 			(remove_unused_layers no)
-			(net 36 "Net-(AOP1-OUT)")
+			(net 35 "Net-(AOP1-OUT)")
 			(pintype "passive")
 		)
@@
 			(layers "*.Cu" "*.Mask")
 			(remove_unused_layers no)
-			(net 32 "R2")
+			(net 34 "Net-(Pot_Digital1-PA0)")
 			(pinfunction "PA0")
 			(pintype "passive")
@@
 			(layers "*.Cu" "*.Mask")
 			(remove_unused_layers no)
-			(net 13 "unconnected-(Pot_Digital1-PW0-Pad6)")
+			(net 34 "Net-(Pot_Digital1-PA0)")
 			(pinfunction "PW0")
-			(pintype "no_connect")
+			(pintype "passive")
 			(solder_mask_margin 0.102)
 		)
@@
 			(layers "*.Cu" "*.Mask")
 			(remove_unused_layers no)
-			(net 1 "GND")
+			(net 32 "R2")
 			(pinfunction "PB0")
 			(pintype "passive")
@@
 			(layers "*.Cu" "*.Mask")
 			(remove_unused_layers no)
-			(net 32 "R2")
+			(net 13 "VCC")
 			(pinfunction "VDD")
 			(pintype "power_in")
@@
 			)
 		)
-		(property "Datasheet" "~"
+		(property "Datasheet" ""
 			(at 0 0 0)
 			(layer "F.Fab")
@@
 			(layers "*.Cu" "*.Mask")
 			(remove_unused_layers no)
-			(net 36 "Net-(AOP1-OUT)")
+			(net 35 "Net-(AOP1-OUT)")
 			(pintype "passive")
 		)
@@
 			)
 		)
-		(property "Datasheet" "~"
+		(property "Datasheet" ""
 			(at 0 0 0)
 			(layer "F.Fab")
@@
 			(layers "*.Cu" "*.Mask")
 			(remove_unused_layers no)
-			(net 36 "Net-(AOP1-OUT)")
+			(net 35 "Net-(AOP1-OUT)")
 			(pintype "passive")
 		)
@@
 			)
 		)
-		(property "Datasheet" "~"
+		(property "Datasheet" ""
 			(at 0 0 0)
 			(layer "F.Fab")

Commit message: flex_sensor
Parts:
- added Flex_sensor1: ~, graphite_emprunts:Flex, F.Cu at (115.2, 59.6)
- added Rflex1: 23k, Resistor_THT:R_Axial_DIN0207_L6.3mm_D2.5mm_P10.16mm_Horizontal, F.Cu at (113.8, 55.5)
Connections:
- J3 pad 2: /A1 -> Flex
- Pot_Digital1 pad 5: Net-(Pot_Digital1-PA0) -> GND
- Pot_Digital1 pad 6: Net-(Pot_Digital1-PA0) -> GND
